File: UWSC_PCB/UWSC_PCB.kicad_pcb (KiCad board)
At the start: 2 copper layers, 8 parts, among them Q1 IRF1405, Q2 IRF1405, U1 IR2101

Commit message: update
Parts:
- added C2: C_Polarized, Capacitor_THT:CP_Radial_D4.0mm_P2.00mm, F.Cu at (151.5, 67.1)
- added C4: CAPACITOR, Capacitor_THT:CP_Radial_D4.0mm_P2.00mm, F.Cu at (151.5, 78.2)
- added C5: C_Polarized, Capacitor_THT:CP_Radial_D4.0mm_P2.00mm, F.Cu at (151.5, 83.7)
- added C6: CAPACITOR, Capacitor_THT:CP_Radial_D4.0mm_P2.00mm, F.Cu at (151.5, 89.3)
- added D2: D, Diode_SMD:D_0201_0603Metric, F.Cu at (187.2, 74.2)
- added D3: D, Diode_SMD:D_0201_0603Metric, F.Cu at (188.4, 71.8)
- added Q3: IRF1405, IRF1405:TO254P483X1016X1994-3P, F.Cu at (169.7, 74.2)
- added Q4: IRF1405, IRF1405:TO254P483X1016X1994-3P, F.Cu at (158.9, 75.7)
- added Q5: IRF1405, IRF1405:TO254P483X1016X1994-3P, F.Cu at (158.9, 82.1)
- added Q6: IRF1405, IRF1405:TO254P483X1016X1994-3P, F.Cu at (158.9, 88.5)
- added R3: R, Resistor_SMD:R_0201_0603Metric, F.Cu at (186.6, 86.7)
- added R4: R, Resistor_SMD:R_0201_0603Metric, F.Cu at (186.6, 88.4)
- added R5: R, Resistor_SMD:R_0201_0603Metric, F.Cu at (186.6, 90.2)
- added R6: R, Resistor_SMD:R_0201_0603Metric, F.Cu at (186.6, 91.9)
- added U2: ATMEGA328P-AU, digikey-footprints:TQFP-32_7x7mm, F.Cu at (179.6, 88.0)
- added U3: IR2101, Package_DIP:DIP-8_W7.62mm_SMDSocket_SmallPads, F.Cu at (179.8, 76.5)
- added U4: IR2101, Package_DIP:DIP-8_W7.62mm_SMDSocket_SmallPads, F.Cu at (185.1, 64.7)
- moved C3 31.9 mm to (151.5, 72.6)
- moved Q2 28.7 mm to (158.9, 69.3), turned to 0 degrees
- moved R1 28.3 mm to (186.6, 83.2), turned to 0 degrees
- moved U1 17.2 mm to (173.4, 64.7)
- moved C1 15.0 mm to (151.5, 61.5), turned to 0 degrees
- moved Q1 13.9 mm to (158.9, 63.0)
- moved D1 10.8 mm to (186.6, 72.1), turned to -90 degrees
- moved R2 10.5 mm to (186.6, 84.9)

Commit message: update
Parts:
- moved U2 75.9 mm to (128.8, 31.6)
- moved U1 54.1 mm to (154.7, 14.0)
- moved C2 53.5 mm to (174.0, 18.5)
- moved C1 53.2 mm to (144.3, 8.89)
- moved C3 52.8 mm to (180.9, 28.7)
- moved Q1 45.5 mm to (164.1, 17.8)
- moved Q2 44.6 mm to (169.2, 25.9)
- moved Q6 40.9 mm to (138.4, 53.1), turned to 180 degrees
- moved U3 39.2 mm to (177.8, 37.3), turned to 0 degrees
- moved C4 36.0 mm to (178.6, 54.4)
- moved C6 34.4 mm to (143.3, 55.9)
- moved Q5 32.8 mm to (133.3, 61.5)
- moved U4 32.7 mm to (152.4, 63.2)
- moved Q4 30.0 mm to (172.5, 49.0)
- moved D1 28.3 mm to (164.3, 54.6)
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Other:
- board outline added: 68 x 68 mm
